Commit message: Update urdf in spotmicro pybullet

File: OpenQuad_V2/yellow_ros/src/spotmicro/util/pybullet_data/assets/yellow_urdf/yellow_spot.urdf (robot description, URDF)
Before this commit: robot spot, 24 links, 23 joints
Links:
- link back: mass 0.1 -> 0.116; geometry collision box size=0.114 0.117 0.091; visual mesh filename=package://mini_ros/yellow_stl/back_cover_v2.stl scale=0.001 0.001 0.001
- link back_bracket: mass 0.1 -> 0.153; geometry collision box size=0.11 0.104 0.092; visual mesh filename=package://mini_ros/yellow_stl/back_plate_v2.stl scale=0.001 0.001 0.001
- link back_left_foot: mass 0.005 -> 0.009
- link back_left_hip: mass 0.2 -> 0.209; geometry collision box size=0.05 0.072 0.072; visual mesh filename=package://mini_ros/yellow_stl/LEFT_HIP.stl scale=0.001 0.001 0.001
- link back_left_lower_leg: mass 0.05 -> 0.036; geometry collision box size=0.022 0.034 0.155; visual mesh filename=package://mini_ros/yellow_stl/LEFT_LOWER_LEG.stl scale=0.001 0.001 0.001
- link back_left_upper_leg: mass 0.13 -> 0.268; geometry collision box size=0.081 0.068 0.169; visual mesh filename=package://mini_ros/yellow_stl/LEFT_UPPER_LEG.stl scale=0.001 0.001 0.001
- link back_right_foot: mass 0.005 -> 0.009
- link back_right_hip: mass 0.2 -> 0.209; geometry collision box size=0.05 0.072 0.072; visual mesh filename=package://mini_ros/yellow_stl/RIGHT_HIP.stl scale=0.001 0.001 0.001
- link back_right_lower_leg: mass 0.05 -> 0.036; geometry collision box size=0.022 0.034 0.155; visual mesh filename=package://mini_ros/yellow_stl/RIGHT_LOWER_LEG.stl scale=0.001 0.001 0.001
- link back_right_upper_leg: mass 0.13 -> 0.268; geometry collision box size=0.081 0.068 0.169; visual mesh filename=package://mini_ros/yellow_stl/RIGHT_UPPER_LEG.stl scale=0.001 0.001 0.001
- link base_inertia: geometry collision box size=0.114 0.232 0.145; visual mesh filename=package://mini_ros/yellow_stl/MAINBODY.stl scale=0.001 0.001 0.001
- link chassis_left: mass 0.01 -> 0.024; geometry collision box size=0.0135 0.1687 0.0414; visual mesh filename=package://mini_ros/yellow_stl/platform_left_side_v2_rescale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 scale=0.001 0.001 0.001
- link chassis_right: mass 0.01 -> 0.024; geometry collision box size=0.0135 0.1687 0.0414; visual mesh filename=package://mini_ros/yellow_stl/platform_right_side_v2_rescal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 scale=0.001 0.001 0.001
- link front: mass 0.1 -> 0.153; geometry collision box size=0.116 0.127 0.103; visual mesh filename=package://mini_ros/yellow_stl/front_cover_v2.stl scale=0.001 0.001 0.001
- link front_bracket: mass 0.1 -> 0.14; geometry collision box size=0.11 0.103 0.092; visual mesh filename=package://mini_ros/yellow_stl/front_plate_v2.stl scale=0.001 0.001 0.001
- link front_left_foot: mass 0.005 -> 0.009
- link front_left_hip: mass 0.2 -> 0.209; geometry collision box size=0.05 0.072 0.072; visual mesh filename=package://mini_ros/yellow_stl/LEFT_HIP.stl scale=0.001 0.001 0.001
- link front_left_lower_leg: mass 0.05 -> 0.036; geometry collision box size=0.022 0.034 0.155; visual mesh filename=package://mini_ros/yellow_stl/LEFT_LOWER_LEG.stl scale=0.001 0.001 0.001
- link front_left_upper_leg: mass 0.13 -> 0.268; geometry collision box size=0.081 0.068 0.169; visual mesh filename=package://mini_ros/yellow_stl/LEFT_UPPER_LEG.stl scale=0.001 0.001 0.001
- link front_right_foot: mass 0.005 -> 0.009
- link front_right_hip: mass 0.2 -> 0.209; geometry collision box size=0.05 0.072 0.072; visual mesh filename=package://mini_ros/yellow_stl/RIGHT_HIP.stl scale=0.001 0.001 0.001
- link front_right_lower_leg: mass 0.05 -> 0.036; geometry collision box size=0.022 0.034 0.155; visual mesh filename=package://mini_ros/yellow_stl/RIGHT_LOWER_LEG.stl scale=0.001 0.001 0.001
- link front_right_upper_leg: mass 0.13 -> 0.268; geometry collision box size=0.081 0.068 0.169; visual mesh filename=package://mini_ros/yellow_stl/RIGHT_UPPER_LEG.stl scale=0.001 0.001 0.001
